Commit message: Correct formulas (robust version, but no sensor-model integration)

File: fmauch_universal_robot/ur_e_description/urdf/ur10e.urdf.xacro (robot description, xacro)
@@ -17,10 +17,10 @@
   </xacro:macro>
   <xacro:macro name="ur10e_robot" params="prefix joint_limited
-    shoulder_pan_lower_limit:=${-pi}    shoulder_pan_upper_limit:=${pi}
-    shoulder_lift_lower_limit:=${-pi}    shoulder_lift_upper_limit:=${pi}
-    elbow_joint_lower_limit:=${-pi}    elbow_joint_upper_limit:=${pi}
-    wrist_1_lower_limit:=${-2*pi}    wrist_1_upper_limit:=${2*pi}
-    wrist_2_lower_limit:=${-2*pi}    wrist_2_upper_limit:=${2*pi}
-    wrist_3_lower_limit:=${-2*pi}    wrist_3_upper_limit:=${2*pi}
+    shoulder_pan_lower_limit:=-3    shoulder_pan_upper_limit:=3
+    shoulder_lift_lower_limit:=-3    shoulder_lift_upper_limit:=0.52
+    elbow_joint_lower_limit:=-2.9    elbow_joint_upper_limit:=0.1
+    wrist_1_lower_limit:=${-pi}    wrist_1_upper_limit:=${pi}
+    wrist_2_lower_limit:=${-pi}    wrist_2_upper_limit:=${pi}
+    wrist_3_lower_limit:=${-pi}    wrist_3_upper_limit:=${pi}
     transmission_hw_interface:=hardware_interface/PositionJointInterface
     safety_limits:=false safety_pos_margin:=0.15
@@ -84,5 +84,5 @@
       </xacro:unless>
       <xacro:if value="${joint_limited}">
-        <limit lower="${shoulder_pan_lower_limit}" upper="${shoulder_pan_upper_limit}" effort="330.0" velocity="1.8"/>
+        <limit lower="${shoulder_pan_lower_limit}" upper="${shoulder_pan_upper_limit}" effort="330.0" velocity="0.01"/>
         <xacro:if value="${safety_limits}">
           <safety_controller soft_lower_limit="${shoulder_pan_lower_limit + safety_pos_margin}" soft_upper_limit="${shoulder_pan_upper_limit - safety_pos_margin}" k_position="${safety_k_position}" k_velocity="0.0"/>

Commit message: Save fine working version Add stitcher-node to work with CoppeliaSim. However, uncertainty is still not considered properly and subject to implementation.

File: fmauch_universal_robot/ur_e_description/urdf/ur10e.urdf.xacro (robot description, xacro)
@@ -17,5 +17,5 @@
   </xacro:macro>
   <xacro:macro name="ur10e_robot" params="prefix joint_limited
-    shoulder_pan_lower_limit:=-3    shoulder_pan_upper_limit:=3
+    shoulder_pan_lower_limit:=-3.14    shoulder_pan_upper_limit:=3.14
     shoulder_lift_lower_limit:=-3    shoulder_lift_upper_limit:=0.52
     elbow_joint_lower_limit:=-2.9    elbow_joint_upper_limit:=0.1

File: fmauch_universal_robot/ur_e_description/urdf/ur10e_joint_limited_robot.urdf.xacro (robot description, xacro)
@@ -69,5 +69,5 @@
     <parent link="tool0"/>
     <child link="scanner_focus"/>
-    <origin xyz="0 1.2500e-01 1.4714e-01" rpy="0 0 1.5707963"/>
+    <origin xyz="0 0.15 0.171" rpy="0 0 1.5707963"/>
   </joint>
  <!--added: END       <origin xyz="${-(0.125/2)-(0.11/2)} -0.01 0" rpy="0 0 ${pi/2}" /> -->
