Commit message: Use map to store scanner params

File: fmauch_universal_robot/ur_e_description/urdf/ur10e_joint_limited_robot.urdf.xacro (robot description, xacro)
@@ -19,10 +19,10 @@
     kinematics_file="${load_yaml('$(arg kinematics_config)')}"
     />
-   <!-- added by Adem: TO DO: create a separate file -->
-  <material name="gray">
+   <!-- added by Adem, modified by Sven -->
+  <material name="white">
     <color rgba="1 1 1 1"/>
   </material>
-  <material name="blue">
-    <color rgba="0 0 1 1"/>
+  <material name="wbk_green">
+    <color rgba="0.0 0.59 0.51 1"/>
   </material>
   <link name="table">
@@ -31,5 +31,5 @@
         <box size="1 1 1.1"/>
       </geometry>
-      <material name="gray"/>
+      <material name="white"/>
     </visual>
   </link>
@@ -39,38 +39,31 @@
     <origin xyz="0.36 0.36 0.55" rpy="0 0 0" />
   </joint>
-  <link name="zivid_camera">
+  <link name="laser_scanner">
     <visual>
       <geometry>
-        <box size="0.23 0.10 0.16"/>
+        <box size="0.15 0.3 0.17"/>
       </geometry>
-      <material name="blue"/>
-      <origin rpy="0 0 0" xyz="0.08 0 -0.075"/>  <!--"0 0 0" xyz="0.08 0 -0.075" -->
+      <material name="wbk_green"/>
+      <origin rpy="0 0 0" xyz="0.00 0.075 0.086"/>  <!--tiny offset to ensure friction-absence -->
     </visual>
     <collision>
-      <origin rpy="0 0 0" xyz="0.08 0 -0.075"/>
+      <origin rpy="0 0 0" xyz="0.0 0.08 0.095"/>
       <geometry>
-        <box size="0.25 0.12 0.18"/>     <!--size="0.23 0.09 0.15" -->
+        <box size="0.17 0.32 0.19"/>     <!--size="0.23 0.09 0.15" -->
       </geometry>
     </collision>
   </link>
-  <link name="camera_halterung">
-    <visual>
-      <geometry>
-        <box size=" 0.11 0.065 0.035"/>
-      </geometry>
-      <material name="blue"/>
-    </visual>
-  </link>
-  <joint name="h_cam" type="fixed">
-    <parent link="camera_halterung"/>
-    <child link="zivid_camera"/>
-    <origin xyz="${-(0.11/2)-(0.085/2) - 0.01} -0.08 0.06" rpy="0 0 ${pi/2}" />
+  <joint name="scanner_connection" type="fixed">
+    <parent link="tool0"/>
+    <child link="laser_scanner"/>
+    <origin xyz="0 0 0" rpy="0.0 0.0 0.0" />
   </joint>
-  <joint name="ee_h" type="fixed">
+  <link name="scanner_focus" ></link>
+  <joint name="scanner_internal" type="fixed">
     <parent link="tool0"/>
-    <child link="camera_halterung"/>
-    <origin xyz="0 -0.031 0.018" rpy="0 0.0 ${pi/2}" />
+    <child link="scanner_focus"/>
+    <origin xyz="0 1.2500e-01 1.4714e-01" rpy="3.1415927 -1.3089969 1.5707963"/>
   </joint>
- <!--added by Adem: END       <origin xyz="${-(0.125/2)-(0.11/2)} -0.01 0" rpy="0 0 ${pi/2}" /> -->
+ <!--added: END       <origin xyz="${-(0.125/2)-(0.11/2)} -0.01 0" rpy="0 0 ${pi/2}" /> -->
   <link name="world" />
   <joint name="world_joint" type="fixed">

Commit message: Update sensor model to latest values

File: fmauch_universal_robot/ur_e_description/urdf/ur10e_joint_limited_robot.urdf.xacro (robot description, xacro)
@@ -45,17 +45,29 @@
     <origin xyz="0.36 0.36 0.55" rpy="0 0 0" />
   </joint>
+  <!-- See corresponding Bachelor Thesis for the origin of these numbers -->
   <link name="laser_scanner">
     <visual>
       <geometry>
-        <box size="0.15 0.3 0.17"/>
+        <mesh scale="0.001 0.001 0.001" filename="package://ur_e_description/meshes/laser_scanner/zeiss_tscan_visual.stl" />
       </geometry>
       <material name="wbk_green"/>
-      <origin rpy="0 0 0" xyz="0.00 0.075 0.086"/>  <!--tiny offset to ensure friction-absence -->
+      <!-- Those parameters have been optimized heuristically so that the visual model is apprx. enclosed by the collision model-->
+      <origin rpy="0 -1.5707963267948966 -1.5707963267948966" xyz="-0.05 0 0.013"/>
     </visual>
+    <!--Body-->
     <collision>
-      <origin rpy="0 0 0" xyz="0.0 0.08 0.095"/>
+      <origin rpy="0 0 0" xyz="0.0 0.0 0.083"/>
       <geometry>
-        <box size="0.17 0.32 0.19"/>     <!--size="0.23 0.09 0.15" -->
+        <box size="0.125 0.052 0.058"/>
       </geometry>
+      <material name="wbk_green"/>
+    </collision>
+    <!--Handle-->
+    <collision>
+      <origin rpy="0 0 0" xyz=" 0.155 0.0 0.09"/>
+      <geometry>
+        <box size="0.185 0.16 0.18"/>     <!--size="0.23 0.09 0.15" -->
+      </geometry>
+      <material name="wbk_green"/>
     </collision>
   </link>
@@ -65,11 +77,10 @@
     <origin xyz="0 0 0" rpy="0.0 0.0 0.0" />
   </joint>
-  <link name="scanner_focus" ></link>
+  <link name="laser_emitter_frame" ></link>
   <joint name="scanner_internal" type="fixed">
-    <parent link="tool0"/>
-    <child link="scanner_focus"/>
-    <origin xyz="0 0.15 0.171" rpy="0 0 1.5707963"/>
+    <parent link="laser_scanner"/>
+    <child link="laser_emitter_frame"/>
+    <origin xyz="0.1665 0.0 0.14318" rpy="0 0 0"/>
   </joint>
- <!--added: END       <origin xyz="${-(0.125/2)-(0.11/2)} -0.01 0" rpy="0 0 ${pi/2}" /> -->
   <link name="world" />
   <joint name="world_joint" type="fixed">

Commit message: Abgabecode

File: fmauch_universal_robot/ur_e_description/urdf/ur10e_joint_limited_robot.urdf.xacro (robot description, xacro)
@@ -30,5 +30,5 @@
     <visual>
       <geometry>
-        <box size="1 1 1.1"/>
+        <box size="1 1 0.9"/>
       </geometry>
       <material name="white"/>
@@ -37,5 +37,5 @@
       <origin rpy="0 0 0" xyz="0.0 0.0 0.0"/>
       <geometry>
-        <box size="1 1 1.1"/>
+        <box size="1 1 0.9"/>
       </geometry>
     </collision>
@@ -44,5 +44,5 @@
     <parent link="table"/>
     <child link="base_link"/>
-    <origin xyz="0.36 0.36 0.55" rpy="0 0 0" />
+    <origin xyz="0.36 0.36 0.45" rpy="0 0 0" />
   </joint>
   <!-- See corresponding Bachelor Thesis for the origin of these numbers / geometries / ... -->
@@ -88,5 +88,5 @@
     <parent link="world" />
     <child link = "table" />
-    <origin xyz="0.5 -0.5 0.55" rpy="0.0 0.0 0.0" />
+    <origin xyz="0.5 -0.5 0.45" rpy="0.0 0.0 0.0" />
   </joint>
 </robot>
