Commit message: Tidy up XACRO-files and introduce more qualified fixture model

File: fmauch_universal_robot/ur_e_description/urdf/endeffector_none.xacro (robot description, xacro)
@@ -20,4 +20,6 @@
     kinematics_file="${load_yaml('$(arg kinematics_config)')}"
     />
+  <!-- add fixture -->
+  <xacro:include filename="$(find ur_e_description)/urdf/ur10e_fixture.urdf.xacro" />
    <!-- added by Adem, modified by Sven -->
   <material name="white">

File: fmauch_universal_robot/ur_e_description/urdf/ur10e_joint_limited_robot.urdf.xacro (robot description, xacro)
@@ -3,4 +3,6 @@
   name="ur10e" >
   <xacro:arg name="transmission_hw_interface" default="hardware_interface/PositionJointInterface"/>
+  <xacro:arg name="endeffector" default="NONE"/>
+  <xacro:property name="endeffector" value="$(arg endeffector)"/>
   <!-- common stuff -->
   <xacro:include filename="$(find ur_e_description)/urdf/common.gazebo.xacro" />
@@ -46,58 +48,18 @@
     <origin xyz="0.36 0.36 0.45" rpy="0 0 0" />
   </joint>
-  <link name="fixture">
-    <visual>
-      <geometry>
-        <mesh scale="0.001 0.001 0.001" filename="package://ur_e_description/meshes/custom/fixture.stl" />
-      </geometry>
-      <material name="white"/>
-    </visual>
-    <collision>
-      <origin rpy="0 0 0" xyz="0.0 0.0 0.0"/>
-      <geometry>
-        <mesh scale="0.001 0.001 0.001" filename="package://ur_e_description/meshes/custom/collision/fixture.stl" />
-      </geometry>
-    </collision>
-  </link>
-  <joint name="table_fixture" type="fixed">
-    <parent link="table"/>
-    <child link="fixture"/>
-    <origin xyz="0.0 -0.24 0.45" rpy="1.570796327 0 0" />
-  </joint>
-  <joint name="tool0_end_effector" type="fixed">
-    <parent link="tool0"/>
-    <child link="end_effector"/>
-    <origin xyz="0.0 0.0 0.0" rpy="0 0 3.141592654"/>
-  </joint>
-  <link name="end_effector">
-    <visual>
-      <geometry>
-        <mesh scale="0.001 0.001 0.001" filename="package://ur_e_description/meshes/custom/zivid_gripper.stl" />
-      </geometry>
-      <material name="end_effector_dark_gray"/>
-      <origin rpy="0 0 0" xyz="0 0 0"/>
-    </visual>
-    <collision>
-      <geometry>
-        <mesh scale="0.001 0.001 0.001" filename="package://ur_e_description/meshes/custom/collision/zivid.stl" />
-      </geometry>
-      <material name="end_effector_dark_gray"/>
-      <origin rpy="0 0 0" xyz="0 0 0"/>
-    </collision>
-    <collision>
-      <geometry>
-        <mesh scale="0.001 0.001 0.001" filename="package://ur_e_description/meshes/custom/collision/zivid_mount.stl" />
-      </geometry>
-      <material name="end_effector_dark_gray"/>
-      <origin rpy="0 0 0" xyz="0 0 0"/>
-    </collision>
-    <collision>
-      <geometry>
-        <box size="0.21 0.04 0.194"/>
-      </geometry>
-      <material name="end_effector_dark_gray"/>
-      <origin rpy="0 0 0" xyz="0 0 0.163"/>
-    </collision>
-  </link>
+  <!-- add fixture -->
+  <xacro:include filename="$(find ur_e_description)/urdf/fixture.xacro" />
+  <!-- Load endeffector config -->
+  <xacro:if value="${endeffector != 'none'}">
+    <xacro:include filename="$(find ur_e_description)/urdf/endeffector_$(arg endeffector).xacro" />
+  </xacro:if>
+  <xacro:if value="${endeffector == 'none'}">
+    <joint name="dummy_joint" type="fixed">
+      <origin xyz="0 0 0" rpy="0 0 0"/>
+      <parent link="tool0"/>
+      <child link="tool_center_point"/>
+    </joint>
+    <link name="tool_center_point"/>
+  </xacro:if>
   <link name="world" />
   <joint name="world_joint" type="fixed">

Commit message: Add new fixture CAD and controller node

File: fmauch_universal_robot/ur_e_description/urdf/endeffector_none.xacro (robot description, xacro)
@@ -2,93 +2,9 @@
 <robot xmlns:xacro="http://ros.org/wiki/xacro"
   name="ur10e" >
-  <xacro:arg name="transmission_hw_interface" default="hardware_interface/PositionJointInterface"/>
-  <!-- common stuff -->
-  <xacro:include filename="$(find ur_e_description)/urdf/common.gazebo.xacro" />
-  <!-- ur10e -->
-  <xacro:include filename="$(find ur_e_description)/urdf/ur10e.urdf.xacro" />
-  <!-- arm -->
-  <xacro:arg name="kinematics_config" default="$(find ur_e_description)/config/ur10e_default.yaml"/>
-  <!-- Use numerical values instead of "pi" to assert coherence with the joint_limits.yaml -->
-  <xacro:ur10e_robot prefix="" joint_limited="true"
-    shoulder_pan_lower_limit="-6.283" shoulder_pan_upper_limit="6.283"
-    shoulder_lift_lower_limit="-3.14"    shoulder_lift_upper_limit="0.52"
-    elbow_joint_lower_limit="-2.9"    elbow_joint_upper_limit="0.1"
-    wrist_1_lower_limit="-6.283"      wrist_1_upper_limit="6.283"
-    wrist_2_lower_limit="-6.283"      wrist_2_upper_limit="6.283"
-    wrist_3_lower_limit="-6.283"      wrist_3_upper_limit="6.283"
-    transmission_hw_interface="$(arg transmission_hw_interface)"
-    kinematics_file="${load_yaml('$(arg kinematics_config)')}"
-    />
-  <!-- add fixture -->
-  <xacro:include filename="$(find ur_e_description)/urdf/ur10e_fixture.urdf.xacro" />
-   <!-- added by Adem, modified by Sven -->
-  <material name="white">
-    <color rgba="1 1 1 1"/>
-  </material>
-  <material name="wbk_green">
-    <color rgba="0.0 0.59 0.51 1"/>
-  </material>
-  <link name="table">
-    <visual>
-      <geometry>
-        <box size="1 1 0.9"/>
-      </geometry>
-      <material name="white"/>
-    </visual>
-    <collision>
-      <origin rpy="0 0 0" xyz="0.0 0.0 0.0"/>
-      <geometry>
-        <box size="1 1 0.9"/>
-      </geometry>
-    </collision>
-  </link>
-  <joint name="table_base" type="fixed">
-    <parent link="table"/>
-    <child link="base_link"/>
-    <origin xyz="0.36 0.36 0.45" rpy="0 0 0" />
+  <joint name="dummy_joint" type="fixed">
+    <origin xyz="0 0 0" rpy="0 0 0"/>
+    <parent link="tool0"/>
+    <child link="tool_center_point"/>
   </joint>
-  <!-- See corresponding Bachelor Thesis for the origin of these numbers / geometries / ... -->
-  <link name="laser_scanner">
-    <visual>
-      <geometry>
-        <mesh scale="0.001 0.001 0.001" filename="package://ur_e_description/meshes/custom/zeiss_tscan_visual.stl" />
-      </geometry>
-      <material name="wbk_green"/>
-      <!-- Those parameters have been optimized heuristically so that the visual model is apprx. enclosed by the collision model-->
-      <origin rpy="0 -1.5707963267948966 -1.5707963267948966" xyz="-0.05 0 0.013"/>
-    </visual>
-    <!--Handle-->
-    <collision>
-      <origin rpy="0 0 0" xyz="0.0 0.0 0.083"/>
-      <geometry>
-        <box size="0.125 0.052 0.058"/>
-      </geometry>
-      <material name="wbk_green"/>
-    </collision>
-    <!--Body-->
-    <collision>
-      <origin rpy="0 0 0" xyz=" 0.155 0.0 0.09"/>
-      <geometry>
-        <box size="0.185 0.16 0.18"/>     <!--size="0.23 0.09 0.15" -->
-      </geometry>
-      <material name="wbk_green"/>
-    </collision>
-  </link>
-  <joint name="scanner_connection" type="fixed">
-    <parent link="tool0"/>
-    <child link="laser_scanner"/>
-    <origin xyz="0 0 0" rpy="0.0 0.0 0.0" />
-  </joint>
-  <link name="laser_emitter_frame" ></link>
-  <joint name="scanner_internal" type="fixed">
-    <parent link="laser_scanner"/>
-    <child link="laser_emitter_frame"/>
-    <origin xyz="0.1665 0.0 0.14318" rpy="0 0 0"/>
-  </joint>
-  <link name="world" />
-  <joint name="world_joint" type="fixed">
-    <parent link="world" />
-    <child link = "table" />
-    <origin xyz="0.5 -0.5 0.45" rpy="0.0 0.0 0.0" />
-  </joint>
+  <link name="tool_center_point"/>
 </robot>

File: fmauch_universal_robot/ur_e_description/urdf/fixture.xacro (robot description, xacro)
@@ -1,18 +1,20 @@
 <?xml version="1.0"?>
 <robot xmlns:xacro="http://ros.org/wiki/xacro">
-  <link name="fixture">
+  <link name="fixture_static">
     <visual>
        <origin xyz="0.0 0.0 0.0" rpy="1.570796327 0 0" />
       <geometry>
-        <mesh scale="0.001 0.001 0.001" filename="package://ur_e_description/meshes/custom/fixture.stl" />
+        <mesh scale="0.001 0.001 0.001" filename="package://ur_e_description/meshes/custom/fixture_static.stl" />
       </geometry>
       <material name="white"/>
     </visual>
+    <!-- Static part of fixture (anvil) -->
     <collision>
-        <origin xyz="0.0 0.00 0.0" rpy="1.570796327 0 0" />
+        <origin xyz="0.17 0.0 0.0975" rpy="0 0 0" />
         <geometry>
-            <mesh scale="0.001 0.001 0.001" filename="package://ur_e_description/meshes/custom/collision/fixture_1.stl" />-->
+            <box size="0.13 0.19 0.165"/>-->
         </geometry>
     </collision>
+    <!-- Static part of fixture (hammer-side)-->
     <collision>
         <origin xyz="-0.215 -0.005 0.125" rpy="0 0 0" />
@@ -23,4 +25,5 @@
         </geometry>
     </collision>
+    <!-- Ground plane -->
     <collision>
         <origin xyz="0.005 0.0 0.0125" rpy="0 0 0" />
@@ -32,6 +35,28 @@
   <joint name="table_fixture" type="fixed">
     <parent link="table"/>
-    <child link="fixture"/>
+    <child link="fixture_static"/>
     <origin xyz="0.0 -0.24 0.45" rpy="0 0 0" />
   </joint>
+  <joint name="fixture_static_dynamic" type="prismatic">
+    <parent link="fixture_static"/>
+    <child link="fixture_dynamic"/>
+    <origin xyz="0.0 0.0 0.0" rpy="0 0 0" />
+    <axis xyz="1.0 0.0 0.0"/>
+    <limit upper="0.186" lower="0.0" effort="10" velocity="10"/>-
+  </joint>
+  <link name="fixture_dynamic">
+    <visual>
+       <origin xyz="0.0 0.0 0.0" rpy="1.570796327 0 0" />
+      <geometry>
+        <mesh scale="0.001 0.001 0.001" filename="package://ur_e_description/meshes/custom/fixture_dynamic.stl" />
+      </geometry>
+      <material name="white"/>
+    </visual>
+    <collision>
+          <origin xyz="-0.204 -0.00225 0.1235" rpy="0 0 0" />
+          <geometry>
+              <box size="0.345 0.115 0.115"/>
+          </geometry>
+      </collision>
+    </link>
 </robot>

File: fmauch_universal_robot/ur_e_description/urdf/ur10e_joint_limited_robot.urdf.xacro (robot description, xacro)
@@ -51,15 +51,5 @@
   <xacro:include filename="$(find ur_e_description)/urdf/fixture.xacro" />
   <!-- Load endeffector config -->
-  <xacro:if value="${endeffector != 'none'}">
-    <xacro:include filename="$(find ur_e_description)/urdf/endeffector_$(arg endeffector).xacro" />
-  </xacro:if>
-  <xacro:if value="${endeffector == 'none'}">
-    <joint name="dummy_joint" type="fixed">
-      <origin xyz="0 0 0" rpy="0 0 0"/>
-      <parent link="tool0"/>
-      <child link="tool_center_point"/>
-    </joint>
-    <link name="tool_center_point"/>
-  </xacro:if>
+  <xacro:include filename="$(find ur_e_description)/urdf/endeffector_$(arg endeffector).xacro" />
   <link name="world" />
   <joint name="world_joint" type="fixed">
